File: photodiode.kicad_sch (KiCad schematic)
At the start: 107 parts, among them J1 UART, J11 Conn_01x03_Pin, J13 Conn_01x02_Pin, J2 Conn_01x05_Pin, J3 Conn_01x06_Pin, J4 Micro_SD_Card, J5 Conn_01x02_Male, J6 TL3360, J7 Conn_01x06_Pin, J8 Conn_01x02_Male, J9 KLS7-1290, P1 USB_C_Plug, Q1 BSS138K, Q18 Si2301CDS, Q2 Si2301CDS, Q3 Si2301CDS, Q4 Si2301CDS, U2 SMF05, U22 LS0505, U23 LS0505, U24 W25Q128JVS, U25 MCP1725T, U3 MCP73855, U4 AP22653, U5 ESP32-S3-WROOM-1, U6 MCP1642D, U8 AP3401

Commit message: boost added
Parts:
- removed D1: SK6812MINI, LED_SMD:LED_SK6812MINI_PLCC4_3.5x3.5mm_P1.75mm, symbol LED:SK6812MINI
- removed D2: LED, LED_SMD:LED_1206_3216Metric, symbol Device:LED
- removed J11: Conn_01x03_Pin, KiCAD_Lib:EKMC1601111, symbol Connector:Conn_01x03_Pin
- added C55: 47uF, Capacitor_SMD:C_0603_1608Metric, symbol Device:C
- added Cfilter: 0.1uF, symbol Device:C
- added Cout1: 0.5uF, symbol Device:C
- added D1: D_Schottky, symbol Device:D_Schottky
- added L3: 6uH, symbol Device:L
- added R33: 100k, Resistor_SMD:R_0402_1005Metric, symbol Device:R
- added Rfilter: 100, symbol Device:R
- added Rprotect: 10, symbol Device:R
- added U1: TPS61390RTER, footprints_TPS61390RTER:RTE0016J-OV-IPC_A, symbol TPS61390RTER:TPS61390RTER
- C3: value 100nF -> 2.2uF; footprint Capacitor_SMD:C_0402_1005Metric -> (none); Footprint1 0402 -> (none); Operating Temperature -55°C ~ 125°C -> (none); Order Digikey -> (none); Order1 JLCPCB -> (none); Package1 0402 -> (none); Part Number 311-1676-1-ND -> (none); Part Number1 C426067 -> (none); Price @1 0.1 -> (none); Price @1k 0.012 -> (none); RoHS ROHS3 -> (none); Voltage 16V -> (none)
- C8: value 100nF -> 1uF; Operating Temperature -55°C ~ 125°C -> (none); Part Number 311-1676-1-ND -> 587-1454-1-ND; Part Number1 C426067 -> C14445; Price @1k 0.012 -> 0.02; RoHS ROHS3 -> (none); Voltage 16V -> 10V
- R3: value 10k -> 1ohm; footprint Resistor_SMD:R_0402_1005Metric -> (none); Footprint1 0402 -> (none); Operating Temperature -55°C ~ 155°C -> (none); Order Digikey -> (none); Order1 JLCPCB -> (none); Package1 0402 -> (none); Part Number 311-10.0KLRCT-ND -> (none); Part Number1 C25744 -> (none); Price @1 0.1 -> (none); Price @1k 0.004 -> (none); RoHS ROHS3 -> (none)
Connections:
- net AmbLight: no longer C3.1, R3.2
- net GND: now also C55.2, Cfilter.2, Cout1.2, U1.16 (AGND), U1.17 (Thermal_Pad), U1.7 (GND); no longer R3.1
- net VDD: now also R3.1, C55.1, L3.1, R33.1, U1.10 (VIN); no longer C8.1
- new net: C3.1, R3.2, U1.15 (AVCC)
- new net: Cout1.1, D1.1 (K), Rfilter.1
- new net: Cfilter.1, Rfilter.2, Rprotect.2
- new net: D1.2 (A), L3.2, U1.8 (SW)
- new net: Rprotect.1, U1.6 (MONIN)
- new net a_iapd: U1.1 (VSP)
- new net apd_bias: U1.5 (APD)
- new net tps_en: C8.1, R33.2, U1.13 (EN)
- new net tps_gain_sel: U1.2 (GAIN)
- new net tps_sample: U1.14 (SAMPLE)
Other:
- note added: "APD BIAS"
- note removed: "Ambient Light Sensor"
- note removed: "LED"
- note removed: "PIR"
- moved on the sheet: C6, C7, H1, H2, H3, H4, J13, J2, J3, J4, J6, J7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

Commit message: after save push
Parts:
- added Ccap, Cmon1, Cmon2: 0.5uF, symbol Device:C
- added Radj, Rdown, Rmon1, Rmon2, Rshort, Rup: 100, symbol Device:R
- U1: order_digikey (none) -> https://www.digikey.com/en/products/detail/texas-instrument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
Connections:
- net GND: now also Ccap.2, Cmon1.1, Cmon2.1, Rdown.2, Rmon1.1, Rmon2.1, Rshort.2
- net at Cout1.1, D1.1 (K), Rfilter.1: now also Rup.1
- net at U1.11 (ISHORT): now also Rshort.1
- net at U1.12 (FB): now also Radj.2, Rdown.1, Rup.2
- net iapd_mon2: now reaches U1.3 (MON2)
- net iapd_mon2: now also Cmon2.2, Rmon2.2
- net iapd_mon1: now reaches U1.4 (MON1)
- net iapd_mon1: now also Cmon1.2, Rmon1.2
- net at U1.9 (CAP): now also Ccap.1
- new net esp_dac_adj: Radj.1
Other:
- moved on the sheet: C1, C10, C11, C12, C13, C15, C16, C17, C18, C19, C2, C20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

Commit message: tia selected and put
Parts:
- added U7: OPA1S2385IDRCT, DRC10_1P65X2P40_TEX, symbol OPA1S2385IDRCT:OPA1S2385IDRCT
Connections:
- net GND: now also U7.11 (EPAD), U7.5 (V-)
- net VDD: now also U7.9 (V+)

Commit message: novo last changes
Parts:
- removed R87, R88, R89, R90: 10k, Resistor_SMD:R_0402_1005Metric, symbol Device:R
- removed U24: W25Q128JVS, Package_SON:WSON-8-1EP_6x5mm_P1.27mm_EP3.4x4mm, symbol Memory_Flash:W25Q128JVS
- added C14, Cf1, Csh1: 20nF, symbol Device:C
- added D2: D_Photo, symbol Device:D_Photo
- added R34, Rf1: 5k, symbol Device:R
- added Rsc1, Rsc2: 0, symbol Device:R
- renumbered Ccap to Ccap1, Cfilter to Cfilter1, Radj to Radj1, Rdown to Rdown1, Rfilter to Rfilter1, Rprotect to Rprotect1, Rshort to Rshort1, Rup to Rup1
Connections:
- net GND: now also U7.4 (+INA), Csh1.1, D2.2 (A)
- net apd_bias: now also R34.1
- net tia_out_pre: now reaches U7.1 (OUTA)
- net tia_out_pre: now also Cf1.2, Rf1.2, Rsc1.1, Rsc2.1
- net ctr_sc: now reaches U7.10 (SC)
- net in_sc: now reaches U7.2 (INS)
- net in_sc: now also Rsc1.2
- net at U7.3 (-INA): now also C14.1, Cf1.1, Rf1.1
- net pin_b: now reaches U7.6 (+INB)
- net pin_b: now also Csh1.2, Rsc2.2
- net nin_b: now reaches U7.7 (-INB)
- net tia_out: now reaches U7.8 (OUTB)
- new net: C14.2, D2.1 (K), R34.2
- no-connect marks 0 -> 20
Other:
- note added: "MAPD"
- note added: "TIA"
- note removed: "Memory"
- moved on the sheet: C1, C10, C11, C12, C13, C15, C16, C17, C18, C19, C2, C20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

Commit message: 11mhz tia is added
Parts:
- Cf1: value 20nF -> 4.7pF
- Rf1: value 5k -> 3.3k
Other:
- moved on the sheet: Cmon1, J13, J2, J3, J7, Rmon2
